File: Electronics/MiAM_PAMI_DCShield/MiAM_PAMI_DCShield.kicad_sch (KiCad schematic)
At the start: 11 parts, among them J1 Conn_02x04_Odd_Even, J10 Conn_01x02_Male, J11 Conn_02x03_Odd_Even, J4 Conn_01x06_Male, J5 Conn_01x06_Male, J6 Screw_Terminal_01x02, J7 Conn_01x02_Male, J8 Conn_01x02_Male, U1 ESP32-DEVKIT-V1, U4 TB6612FNG

Commit message: Faster DC
Parts:
- renumbered J6 to BAT1, J10 to EMGBUT1, J9 to GPIO1, J1 to I2C1, J4 to MOT1, J5 to MOT2, J7 to PSW1, J11 to SRV1, J8 to UART2
Connections:
- net 1Y: now also MOT1.1 (Pin_1); no longer MOT1.6 (Pin_6)
- net 2Y: now also MOT1.6 (Pin_6); no longer MOT1.1 (Pin_1)
Changed lines of the file:
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@@
     (effects (font (size 1.27 1.27)) (justify right bottom))
+  )
+  (label "2Y" (at 229.87 138.43 0) (fields_autoplaced)
+    (effects (font (size 1.27 1.27)) (justify left bottom))
   )
   (label "STBY" (at 205.105 107.95 0) (fields_autoplaced)
@@
     (effects (font (size 1.27 1.27)) (justify left bottom))
   )
-  (label "2Y" (at 229.87 125.73 0) (fields_autoplaced)
-    (effects (font (size 1.27 1.27)) (justify left bottom))
-  )
   (label "EN12" (at 184.785 128.27 180) (fields_autoplaced)
     (effects (font (size 1.27 1.27)) (justify right bottom))
@@
     (effects (font (size 1.27 1.27)) (justify right bottom))
   )
+  (label "1Y" (at 229.87 125.73 0) (fields_autoplaced)
+    (effects (font (size 1.27 1.27)) (justify left bottom))
+  )
   (label "GPIO23" (at 259.08 45.085 0) (fields_autoplaced)
     (effects (font (size 1.27 1.27)) (justify left bottom))
@@
     (effects (font (size 1.27 1.27)) (justify right bottom))
   )
-  (label "1Y" (at 229.87 138.43 0) (fields_autoplaced)
-    (effects (font (size 1.27 1.27)) (justify left bottom))
-  )
   (label "RX2" (at 85.09 97.155 0) (fields_autoplaced)
     (effects (font (size 1.27 1.27)) (justify left bottom))
@@
   (symbol (lib_id "Connector:Conn_01x02_Male") (at 102.235 55.245 0) (unit 1)
     (in_bom yes) (on_board yes) (dnp no) (fields_autoplaced)
-    (property "Reference" "J10" (at 102.87 50.165 0)
+    (property "Reference" "EMGBUT1" (at 102.87 50.165 0)
       (effects (font (size 1.27 1.27)))
     )
@@
       (project "MiAM_PAMI_DCShield"
         (path "/25619b26-f8ce-486a-87c9-e743f43b219f"
-          (reference "J10") (unit 1)
+          (reference "EMGBUT1") (unit 1)
         )
       )
@@
   (symbol (lib_id "Connector:Conn_01x06_Male") (at 253.365 130.81 0) (unit 1)
     (in_bom yes) (on_board yes) (dnp no) (fields_autoplaced)
-    (property "Reference" "J5" (at 254 120.65 0)
+    (property "Reference" "MOT2" (at 254 120.65 0)
       (effects (font (size 1.27 1.27)))
     )
@@
       (project "MiAM_PAMI_DCShield"
         (path "/25619b26-f8ce-486a-87c9-e743f43b219f"
-          (reference "J5") (unit 1)
+          (reference "MOT2") (unit 1)
         )
       )
@@
   (symbol (lib_id "Connector_Generic:Conn_02x03_Odd_Even") (at 225.425 77.47 0) (unit 1)
     (in_bom yes) (on_board yes) (dnp no) (fields_autoplaced)
-    (property "Reference" "J11" (at 226.695 69.215 0)
+    (property "Reference" "SRV1" (at 226.695 69.215 0)
       (effects (font (size 1.27 1.27)))
     )
@@
       (project "MiAM_PAMI_DCShield"
         (path "/25619b26-f8ce-486a-87c9-e743f43b219f"
-          (reference "J11") (unit 1)
+          (reference "SRV1") (unit 1)
         )
       )
@@
   (symbol (lib_id "MiAM_ESP32:Conn_03x04_Male") (at 242.57 34.925 0) (unit 1)
     (in_bom yes) (on_board yes) (dnp no) (fields_autoplaced)
-    (property "Reference" "J9" (at 241.935 34.925 0)
+    (property "Reference" "GPIO1" (at 241.935 34.925 0)
       (effects (font (size 1.27 1.27)))
     )
@@
       (project "MiAM_PAMI_DCShield"
         (path "/25619b26-f8ce-486a-87c9-e743f43b219f"
-          (reference "J9") (unit 1)
+          (reference "GPIO1") (unit 1)
         )
       )
@@
   (symbol (lib_id "Connector:Conn_01x02_Female") (at 55.88 41.91 0) (unit 1)
     (in_bom yes) (on_board yes) (dnp no) (fields_autoplaced)
-    (property "Reference" "J6" (at 57.15 41.91 0)
+    (property "Reference" "BAT1" (at 57.15 41.91 0)
       (effects (font (size 1.27 1.27)) (justify left))
     )
@@
       (project "MiAM_PAMI_DCShield"
         (path "/25619b26-f8ce-486a-87c9-e743f43b219f"
-          (reference "J6") (unit 1)
+          (reference "BAT1") (unit 1)
         )
       )
@@
   (symbol (lib_id "Connector:Conn_01x02_Male") (at 170.815 41.91 0) (unit 1)
     (in_bom yes) (on_board yes) (dnp no) (fields_autoplaced)
-    (property "Reference" "J8" (at 171.45 36.83 0)
+    (property "Reference" "UART2" (at 171.45 36.83 0)
       (effects (font (size 1.27 1.27)))
     )
@@
       (project "MiAM_PAMI_DCShield"
         (path "/25619b26-f8ce-486a-87c9-e743f43b219f"
-          (reference "J8") (unit 1)
+          (reference "UART2") (unit 1)
         )
       )
@@
   (symbol (lib_id "Connector:Conn_01x06_Male") (at 224.79 130.81 0) (unit 1)
     (in_bom yes) (on_board yes) (dnp no) (fields_autoplaced)
-    (property "Reference" "J4" (at 225.425 120.65 0)
+    (property "Reference" "MOT1" (at 225.425 120.65 0)
       (effects (font (size 1.27 1.27)))
     )
@@
       (project "MiAM_PAMI_DCShield"
         (path "/25619b26-f8ce-486a-87c9-e743f43b219f"
-          (reference "J4") (unit 1)
+          (reference "MOT1") (unit 1)
         )
       )
@@
   (symbol (lib_id "Connector_Generic:Conn_02x04_Odd_Even") (at 204.47 40.64 0) (unit 1)
     (in_bom yes) (on_board yes) (dnp no) (fields_autoplaced)
-    (property "Reference" "J1" (at 205.74 31.75 0)
+    (property "Reference" "I2C1" (at 205.74 31.75 0)
       (effects (font (size 1.27 1.27)))
     )
@@
       (project "MiAM_PAMI_DCShield"
         (path "/25619b26-f8ce-486a-87c9-e743f43b219f"
-          (reference "J1") (unit 1)
+          (reference "I2C1") (unit 1)
         )
       )
@@
   (symbol (lib_id "Connector:Conn_01x02_Male") (at 101.6 43.18 0) (unit 1)
     (in_bom yes) (on_board yes) (dnp no)
-    (property "Reference" "J7" (at 100.33 43.1799 0)
+    (property "Reference" "PSW1" (at 100.33 43.1799 0)
       (effects (font (size 1.27 1.27)) (justify right))
     )
@@
       (project "MiAM_PAMI_DCShield"
         (path "/25619b26-f8ce-486a-87c9-e743f43b219f"
-          (reference "J7") (unit 1)
-        )
-      )
+          (reference "PSW1") (unit 1)
+        )
+      )
