File: Electronics/MiAM_PAMI_PowerShield/MiAM_PAMI_PowerShield.kicad_pcb (KiCad board)
At the start: 2 copper layers, 28.7 x 54.7 mm, 8 parts, among them U2 3V3, U3 MT3608, U4 LM7805_TO220, U5 ESP32-DEVKIT-V1

Commit message: Faster DC
Routing:
- net /5V_POWER: track 38.4 -> 40.0 mm
- net +12V: track 49.6 -> 50.8 mm
- net /BAT_READING: track 67.6 -> 66.7 mm
- net /EMERGENCY_BUTTON: track 34.6 -> 35.3 mm
Changed lines of the file:
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@@
   (via (at 109.347 60.198) (size 0.8) (drill 0.4) (layers "F.Cu" "B.Cu") (net 1))
   (segment (start 102.362 98.044) (end 102.362 66.929) (width 1.5) (layer "F.Cu") (net 2))
+  (segment (start 110.322 63.246) (end 110.3695 63.1985) (width 1.5) (layer "F.Cu") (net 2))
   (segment (start 102.362 66.929) (end 106.045 63.246) (width 1.5) (layer "F.Cu") (net 2))
-  (segment (start 106.4768 105.029) (end 106.045 105.029) (width 1.5) (layer "F.Cu") (net 2))
-  (segment (start 110.322 63.246) (end 110.3695 63.1985) (width 1.5) (layer "F.Cu") (net 2))
-  (segment (start 104.394 103.378) (end 104.394 100.076) (width 1.5) (layer "F.Cu") (net 2))
+  (segment (start 104.013 105.029) (end 104.013 99.695) (width 1.5) (layer "F.Cu") (net 2))
+  (segment (start 104.013 99.695) (end 102.362 98.044) (width 1.5) (layer "F.Cu") (net 2))
+  (segment (start 106.4768 105.029) (end 104.013 105.029) (width 1.5) (layer "F.Cu") (net 2))
   (segment (start 106.045 63.246) (end 110.322 63.246) (width 1.5) (layer "F.Cu") (net 2))
-  (segment (start 104.394 100.076) (end 102.362 98.044) (width 1.5) (layer "F.Cu") (net 2))
-  (segment (start 106.045 105.029) (end 104.394 103.378) (width 1.5) (layer "F.Cu") (net 2))
-  (segment (start 104.902 106.299) (end 107.569 106.299) (width 0.25) (layer "F.Cu") (net 3))
+  (segment (start 100.076 67.326) (end 100.076 98.425) (width 0.25) (layer "F.Cu") (net 3))
+  (segment (start 100.076 98.425) (end 102.616 100.965) (width 0.25) (layer "F.Cu") (net 3))
+  (segment (start 107.569 106.299) (end 108.458 105.41) (width 0.25) (layer "F.Cu") (net 3))
   (segment (start 108.458 105.41) (end 108.458 103.189) (width 0.25) (layer "F.Cu") (net 3))
-  (segment (start 100.076 65.389) (end 100.076 98.425) (width 0.25) (layer "F.Cu") (net 3))
-  (segment (start 100.076 98.425) (end 102.616 100.965) (width 0.25) (layer "F.Cu") (net 3))
+  (segment (start 102.616 100.965) (end 102.616 105.664) (width 0.25) (layer "F.Cu") (net 3))
+  (segment (start 108.458 103.189) (end 110.3695 101.2775) (width 0.25) (layer "F.Cu") (net 3))
+  (segment (start 107.934 59.468) (end 100.076 67.326) (width 0.25) (layer "F.Cu") (net 3))
+  (segment (start 102.616 105.664) (end 103.251 106.299) (width 0.25) (layer "F.Cu") (net 3))
   (segment (start 107.934 59.468) (end 107.934 57.531) (width 0.25) (layer "F.Cu") (net 3))
-  (segment (start 102.616 104.013) (end 104.902 106.299) (width 0.25) (layer "F.Cu") (net 3))
-  (segment (start 107.569 106.299) (end 108.458 105.41) (width 0.25) (layer "F.Cu") (net 3))
-  (segment (start 100.076 65.389) (end 107.934 57.531) (width 0.25) (layer "F.Cu") (net 3))
   (segment (start 105.934 61.468) (end 107.934 59.468) (width 0.25) (layer "F.Cu") (net 3))
-  (segment (start 108.458 103.189) (end 110.3695 101.2775) (width 0.25) (layer "F.Cu") (net 3))
-  (segment (start 102.616 100.965) (end 102.616 104.013) (width 0.25) (layer "F.Cu") (net 3))
-  (segment (start 96.393 79.681) (end 84.9695 68.2575) (width 1) (layer "F.Cu") (net 4))
-  (segment (start 96.393 97.155) (end 96.393 79.681) (width 1) (layer "F.Cu") (net 4))
-  (segment (start 101.092 101.854) (end 96.393 97.155) (width 1) (layer "F.Cu") (net 4))
-  (via (at 101.092 101.854) (size 0.8) (drill 0.4) (layers "F.Cu" "B.Cu") (net 4))
-  (segment (start 106.4768 99.949) (end 102.997 99.949) (width 1) (layer "B.Cu") (net 4))
-  (segment (start 102.997 99.949) (end 101.092 101.854) (width 1) (layer "B.Cu") (net 4))
+  (segment (start 103.251 106.299) (end 107.569 106.299) (width 0.25) (layer "F.Cu") (net 3))
+  (segment (start 96.393 77.216) (end 87.4345 68.2575) (width 1) (layer "F.Cu") (net 4))
+  (segment (start 87.4345 68.2575) (end 84.9695 68.2575) (width 1) (layer "F.Cu") (net 4))
+  (segment (start 96.393 97.155) (end 96.393 77.216) (width 1) (layer "F.Cu") (net 4))
+  (segment (start 99.187 99.949) (end 96.393 97.155) (width 1) (layer "F.Cu") (net 4))
+  (via (at 99.187 99.949) (size 0.8) (drill 0.4) (layers "F.Cu" "B.Cu") (net 4))
+  (segment (start 99.187 99.949) (end 106.4768 99.949) (width 1) (layer "B.Cu") (net 4))
+  (segment (start 99.441 57.785) (end 94.0275 63.1985) (width 1.5) (layer "F.Cu") (net 5))
   (segment (start 102.235 57.785) (end 105.68 57.785) (width 0.25) (layer "F.Cu") (net 5))
-  (segment (start 101.6 57.785) (end 96.1865 63.1985) (width 1.5) (layer "F.Cu") (net 5))
+  (segment (start 94.0275 63.1985) (end 84.9695 63.1985) (width 1.5) (layer "F.Cu") (net 5))
+  (segment (start 102.235 57.785) (end 99.441 57.785) (width 1.5) (layer "F.Cu") (net 5))
   (segment (start 105.68 57.785) (end 105.934 57.531) (width 0.25) (layer "F.Cu") (net 5))
-  (segment (start 102.235 57.785) (end 101.6 57.785) (width 1.5) (layer "F.Cu") (net 5))
-  (segment (start 96.1865 63.1985) (end 84.9695 63.1985) (width 1.5) (layer "F.Cu") (net 5))
   (segment (start 104.648 77.851) (end 107.6526 74.8464) (width 1.5) (layer "F.Cu") (net 6))
-  (segment (start 104.648 93.98) (end 104.648 77.851) (width 1.5) (layer "F.Cu") (net 6))
+  (segment (start 104.648 95.25) (end 104.648 77.851) (width 1.5) (layer "F.Cu") (net 6))
+  (segment (start 107.6526 74.8464) (end 107.6526 66.167) (width 1.5) (layer "F.Cu") (net 6))
   (segment (start 108.0811 65.7385) (end 110.3695 65.7385) (width 1.5) (layer "F.Cu") (net 6))
   (segment (start 107.6526 66.167) (end 108.0811 65.7385) (width 1.5) (layer "F.Cu") (net 6))
-  (segment (start 106.766 95.25) (end 105.918 95.25) (width 1.5) (layer "F.Cu") (net 6))
-  (segment (start 105.918 95.25) (end 104.648 93.98) (width 1.5) (layer "F.Cu") (net 6))
-  (segment (start 107.6526 74.8464) (end 107.6526 66.167) (width 1.5) (layer "F.Cu") (net 6))
-  (segment (start 84.9695 65.7385) (end 85.017 65.786) (width 1) (layer "F.Cu") (net 7))
+  (segment (start 106.766 95.25) (end 104.648 95.25) (width 1.5) (layer "F.Cu") (net 6))
+  (segment (start 98.806 85.852) (end 98.552 85.598) (width 1) (layer "F.Cu") (net 7))
+  (segment (start 88.265 65.786) (end 85.017 65.786) (width 1) (layer "F.Cu") (net 7))
   (segment (start 106.766 90.17) (end 106.766 85.938) (width 1) (layer "F.Cu") (net 7))
-  (segment (start 85.017 65.786) (end 88.265 65.786) (width 1) (layer "F.Cu") (net 7))
-  (segment (start 88.265 65.786) (end 98.552 76.073) (width 1) (layer "F.Cu") (net 7))
-  (segment (start 98.552 76.073) (end 98.552 82.931) (width 1) (layer "F.Cu") (net 7))
+  (segment (start 85.017 65.786) (end 84.9695 65.7385) (width 1) (layer "F.Cu") (net 7))
+  (segment (start 98.552 76.073) (end 88.265 65.786) (width 1) (layer "F.Cu") (net 7))
+  (segment (start 98.552 85.598) (end 98.552 76.073) (width 1) (layer "F.Cu") (net 7))
   (segment (start 106.766 85.938) (end 106.68 85.852) (width 1) (layer "F.Cu") (net 7))
-  (via (at 98.552 82.931) (size 0.8) (drill 0.4) (layers "F.Cu" "B.Cu") (net 7))
-  (segment (start 101.473 85.852) (end 106.68 85.852) (width 1) (layer "B.Cu") (net 7))
-  (segment (start 98.552 82.931) (end 101.473 85.852) (width 1) (layer "B.Cu") (net 7))
+  (via (at 98.806 85.852) (size 0.8) (drill 0.4) (layers "F.Cu" "B.Cu") (net 7))
+  (segment (start 98.806 85.852) (end 106.68 85.852) (width 1) (layer "B.Cu") (net 7))
   (zone (net 1) (net_name "GND") (layer "B.Cu") (hatch edge 0.5)
     (connect_pads (clearance 0.508))
