File: Electronics/MiAM_PAMI_V3_Stepper/MiAM_PAMI_V3_Stepper.kicad_pcb (KiCad board)
At the start: 2 copper layers, 64 x 95 mm, 32 parts, among them J2 Conn_01x03_Male, J3 Conn_01x03_Male, SW1 SW_DPDT_x2, U1 ESP32-DEVKITC-32U, U2 3V3, U3 MT3608, U4 3V3

Commit message: Fix PCB for v3
Parts:
- removed I2C1: Conn_02x04_Odd_Even, Connector_PinHeader_2.54mm:PinHeader_2x04_P2.54mm_Vertical
- removed U6, U7: ~, Connector_PinHeader_2.54mm:PinHeader_1x06_P2.54mm_Vertical
- added D1: LED, LED_THT:LED_D3.0mm, F.Cu at (134.0, 69.8)
- added D2: D_Schottky, Diode_SMD:D_SOD-323_HandSoldering, F.Cu at (160.3, 55.1)
- added J1: TCRT5000L_Breakout, MiAM_ESP32_Footprints:TCRT5000L_Breakout, B.Cu at (124.5, 130.6)
- added J4: TCRT5000L_Breakout, MiAM_ESP32_Footprints:TCRT5000L_Breakout, B.Cu at (148.3, 130.6)
- added J5: TCRT5000L_Breakout, MiAM_ESP32_Footprints:TCRT5000L_Breakout, B.Cu at (172.1, 130.6)
- added R4: 200, Resistor_SMD:R_0805_2012Metric, F.Cu at (128.9, 69.8)
- J2: moved to B.Cu
- J3: value Conn_01x03_Male -> SSD1306_vertical; footprint MiAM_ESP32_Footprints:Microruptor -> MiAM_ESP32_Footprints:SSD1306_vertical; moved to F.Cu
- MOT1, MOT2: footprint Connector_PinHeader_2.54mm:PinHeader_1x04_P2.54mm_Vertical -> Connector_JST:JST_SH_BM04B-SRSS-TB_1x04-1MP_P1.00mm_Vertical; moved to B.Cu
- MS1, MS2, MS3: value SolderJumper_2_Open -> SolderJumper_2_Bridged; footprint Jumper:SolderJumper-2_P1.3mm_Open_RoundedPad1.0x1.5mm -> Jumper:SolderJumper-2_P1.3mm_Bridged_RoundedPad1.0x1.5mm
- U2, U4: value 3V3 -> 5V
- moved J3 63.8 mm to (128.7, 81.0), turned to 0 degrees
- moved J2 42.9 mm to (174.4, 133.3)
- moved EMGBUT1 37.4 mm to (132.7, 57.2)
- moved BAT1 36.9 mm to (168.9, 53.4), turned to -90 degrees
- moved R3 33.8 mm to (132.7, 49.5), turned to 0 degrees
- moved U2 30.1 mm to (150.5, 64.1), turned to 0 degrees
- moved SRV1 23.6 mm to (172.8, 72.6), turned to -90 degrees
- moved R2 23.5 mm to (159.8, 77.5), turned to -90 degrees
- moved U5 23.5 mm to (144.5, 135.9), turned to 90 degrees
- moved R1 22.7 mm to (159.8, 73.0), turned to -90 degrees
- moved GPIO2 17.9 mm to (116.2, 74.9)
- moved U3 13.2 mm to (149.2, 85.7)
- moved U4 7.62 mm to (170.4, 87.9), turned to -90 degrees
- moved MOT2 5.91 mm to (140.5, 121.4), turned to 0 degrees
- moved UART1 5.85 mm to (134.0, 74.9)
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Connections:
- A1 pad 8: /EMERGENCY_BUTTON -> +12V
- A2 pad 8: /EMERGENCY_BUTTON -> +12V
- C3 pad 1: /EMERGENCY_BUTTON -> +12V
- C4 pad 1: /EMERGENCY_BUTTON -> +12V
- EMGBUT1 pad 1: +12V -> /EMERGENCY_BUTTON
- EMGBUT1 pad 2: /EMERGENCY_BUTTON -> /BATTERY_INPUT
- GPIO2 pad 2: /GPIO4 -> /GPIO12
- GPIO2 pad 3: /GPIO12 -> /GPIO15
- J3 pad 1: /GPIO15 -> /SDA
- J3 pad 2: GND -> /SCL
- J3 pad 3: unconnected-(J3-Pin_3-Pad3) -> +3V3
- SRV1 pad 5: /SERVO_PWM_1 -> /SERVO_PWM_2
- SRV1 pad 6: /SERVO_PWM_2 -> /SERVO_PWM_1
- U1 pad 19: unconnected-(U1-EXT_5V-Pad19) -> Net-(D2-K)
- U1 pad 26: /GPIO4 -> /NOT_MOT_EN
- U1 pad 37: /GPIO23 -> /DIR_2
- U1 pad 4: GND -> /TCRT1
- U1 pad 7: /DIR_2 -> /TCRT0
- U1 pad 8: /NOT_MOT_EN -> /TCRT2
- U2 pad 1: +3V3 -> /5V_BOARD
- U2 pad 3: +12V -> /POWER_SWITCH
- U3 pad 1: /POWER_SWITCH -> /EMERGENCY_BUTTON
- U4 pad 3: /EMERGENCY_BUTTON -> +12V
- U5 pad 6: /GPIO2 -> unconnected-(U5-XSHUT-Pad6)
Routing:
- net /GPIO15: track 88.7 -> 0.00 mm, vias 4 -> 0
- net /TCRT2: track 0.00 -> 86.2 mm, vias 0 -> 4
- net /EMERGENCY_BUTTON: track 129.4 -> 44.1 mm
- net /TCRT0: track 0.00 -> 77.9 mm, vias 0 -> 4
- net /GPIO2: track 93.4 -> 16.9 mm, vias 6 -> 0
- net /NOT_MOT_EN: track 0.00 -> 75.9 mm, vias 0 -> 3
- net /GPIO23: track 65.7 -> 0.00 mm, vias 6 -> 0
- net /TCRT1: track 0.00 -> 59.8 mm, vias 0 -> 4
- net /DIR_2: track 61.6 -> 12.2 mm, vias 4 -> 0
- net /STEP_1: track 0.00 -> 48.6 mm, vias 0 -> 4
- net /SDA: track 124.6 -> 78.4 mm, vias 6 -> 4
- net +3V3: track 149.3 -> 190.2 mm, vias 9 -> 7
- net /DIR_1: track 0.00 -> 40.6 mm, vias 0 -> 4
- net /BATTERY_INPUT: track 28.1 -> 65.0 mm
- net +12V: track 41.3 -> 73.6 mm
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Other:
- board text added: "25"
- board text added: "26"
- board text added: "G"
- board text added: "MiAM PAMI Stepper V3 11/2023"
- board text added: "S"
- board text added: "V"
- board text removed: "MiAM PAMI Stepper board 11/2023"

Commit message: Fix pcb v3
Parts:
- C3, C4: footprint Capacitor_THT:CP_Radial_D4.0mm_P2.00mm -> Capacitor_THT:CP_Radial_D6.3mm_P2.50mm
- MS1, MS2, MS3: moved to F.Cu
- moved GPIO2 18.7 mm to (107.4, 58.4)
- moved C3 14.0 mm to (159.0, 120.2), turned to -90 degrees
- moved MOT2 12.3 mm to (141.7, 109.2), turned to 180 degrees
- moved MOT1 12.3 mm to (160.1, 109.2), turned to 180 degrees
- moved MS1 9.87 mm to (137.7, 99.7), turned to 90 degrees
- moved MS2 9.87 mm to (133.9, 99.7), turned to 90 degrees
- moved MS3 9.87 mm to (130.1, 99.7), turned to 90 degrees
- moved C4 1.79 mm to (146.3, 121.2)
- moved J3 1.14 mm to (129.9, 81.0)
- moved UART1 0.89 mm to (134.9, 74.9)
Connections:
- EMGBUT1 pad 2: /BATTERY_INPUT -> /POWER_SWITCH
- MOT1 pad 1: Net-(A1-1B) -> Net-(A1-2B)
- MOT1 pad 2: Net-(A1-1A) -> Net-(A1-2A)
- MOT1 pad 3: Net-(A1-2A) -> Net-(A1-1A)
- MOT1 pad 4: Net-(A1-2B) -> Net-(A1-1B)
- MOT2 pad 1: Net-(A2-1B) -> Net-(A2-2B)
- MOT2 pad 2: Net-(A2-1A) -> Net-(A2-2A)
- MOT2 pad 3: Net-(A2-2A) -> Net-(A2-1A)
- MOT2 pad 4: Net-(A2-2B) -> Net-(A2-1B)
Routing:
- net /BATTERY_INPUT: track 65.0 -> 24.1 mm
- net /POWER_SWITCH: track 21.3 -> 60.2 mm
- net +3V3: track 190.2 -> 208.1 mm, vias 7 -> 4
- net /MS2: track 32.6 -> 39.0 mm
- net /DIR_2: track 12.2 -> 18.1 mm
- net /STEP_2: track 50.3 -> 56.0 mm, vias 0 -> 1
- net /MS3: track 34.5 -> 36.9 mm
- net +12V: track 73.6 -> 71.2 mm
- net /NOT_MOT_EN: track 75.9 -> 73.9 mm
- net Net-(A2-2A): track 4.78 -> 6.42 mm
- net Net-(A2-1A): track 5.41 -> 7.06 mm
- net Net-(A1-2A): track 5.36 -> 7.00 mm
- net Net-(A1-1A): track 4.72 -> 6.37 mm
- net /MS1: track 33.9 -> 35.5 mm
- net /SDA: track 78.4 -> 77.4 mm
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Other:
- board size 64 x 95 mm -> 62 x 95 mm

Commit message: PCB order 2023-11-29
Parts:
- removed GPIO2: Conn_01x07_Male, Connector_PinHeader_2.54mm:PinHeader_1x07_P2.54mm_Vertical
- removed R3: 10k, Resistor_SMD:R_0805_2012Metric_Pad1.20x1.40mm_HandSolder
- added J6: Conn_01x02_Pin, Connector_PinHeader_2.54mm:PinHeader_1x02_P2.54mm_Vertical, F.Cu at (160.3, 84.6)
- added J7: Conn_01x02_Pin, Connector_PinHeader_2.54mm:PinHeader_1x02_P2.54mm_Vertical, F.Cu at (129.5, 74.9)
- added J8: Conn_01x02_Pin, Connector_PinHeader_2.54mm:PinHeader_1x02_P2.54mm_Vertical, F.Cu at (128.5, 60.7)
- added J9: Conn_01x01_Pin, Connector_PinHeader_2.54mm:PinHeader_1x01_P2.54mm_Vertical, F.Cu at (173.0, 67.8)
- MS1, MS2, MS3: value SolderJumper_2_Bridged -> SolderJumper_2_Open; footprint Jumper:SolderJumper-2_P1.3mm_Bridged_RoundedPad1.0x1.5mm -> Jumper:SolderJumper-2_P1.3mm_Open_RoundedPad1.0x1.5mm
Connections:
- EMGBUT1 pad 3: Net-(EMGBUT1-Pin_3) -> GND
Routing:
- net /TCRT2: track 86.1 -> 58.4 mm, vias 4 -> 0
- net /GPIO0: track 0.00 -> 14.8 mm
- net /GPIO18: track 0.00 -> 11.2 mm
- net /GPIO5: track 98.3 -> 87.2 mm
- net /GPIO12: track 0.00 -> 10.2 mm
- net /GPIO15: track 0.00 -> 9.47 mm
- net /GPIO19: track 0.00 -> 9.42 mm
- net +3V3: track 208.1 -> 199.5 mm, vias 4 -> 2
- net /TCRT1: track 60.2 -> 67.9 mm, vias 4 -> 2
- net Net-(EMGBUT1-Pin_3): track 4.13 -> 0.00 mm
- net /GPIO35: track 0.00 -> 3.58 mm
- net /GPIO34: track 0.00 -> 3.58 mm
- net /NOT_MOT_EN: track 73.9 -> 70.4 mm
- net /STEP_1: track 49.0 -> 51.6 mm, vias 4 -> 3
- net Net-(A2-~{RESET}): track 0.00 -> 2.54 mm
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Other:
- board text added: "0"
- board text added: "12"
- board text added: "15"
- board text added: "18"
- board text added: "19"
- board text added: "34"
- board text added: "35"
- board text added: "3V3"
- board text added: "OFF"
- board text added: "ON"
- board text added: "SCL"
- board text added: "SDA"
