File: Electronics/MiAM_PAMI_V3_Stepper/MiAM_PAMI_V3_Stepper.kicad_sch (KiCad schematic)
At the start: 32 parts, among them J2 Conn_01x03_Male, J3 Conn_01x03_Male, SW1 SW_DPDT_x2, U1 ESP32-DEVKITC-32U, U2 3V3, U3 MT3608, U4 3V3

Commit message: Fix PCB for v3
Parts:
- removed I2C1: Conn_02x04_Odd_Even, Connector_PinHeader_2.54mm:PinHeader_2x04_P2.54mm_Vertical, symbol Connector_Generic:Conn_02x04_Odd_Even
- removed J3: Conn_01x03_Male, MiAM_ESP32_Footprints:Microruptor, symbol Connector:Conn_01x03_Male
- removed U6, U7: ~, Connector_PinHeader_2.54mm:PinHeader_1x06_P2.54mm_Vertical, symbol MiAM_ESP32:VL53L01XV2
- added D1: LED, LED_THT:LED_D3.0mm, symbol Device:LED
- added D2: D_Schottky, Diode_SMD:D_SOD-323_HandSoldering, symbol Device:D_Schottky
- added J1, J4, J5: TCRT5000L_Breakout, MiAM_ESP32_Footprints:TCRT5000L_Breakout, symbol MiAM_ESP32:TCRT5000L_Breakout
- added J3: SSD1306_vertical, MiAM_ESP32_Footprints:SSD1306_vertical, symbol MiAM_ESP32:SSD1306_vertical
- added R4: 200, Resistor_SMD:R_0805_2012Metric, symbol Device:R
- MOT1, MOT2: footprint Connector_PinHeader_2.54mm:PinHeader_1x04_P2.54mm_Vertical -> Connector_JST:JST_SH_BM04B-SRSS-TB_1x04-1MP_P1.00mm_Vertical
- MS1, MS2, MS3: value SolderJumper_2_Open -> SolderJumper_2_Bridged; footprint Jumper:SolderJumper-2_P1.3mm_Open_RoundedPad1.0x1.5mm -> Jumper:SolderJumper-2_P1.3mm_Bridged_RoundedPad1.0x1.5mm; symbol Jumper:SolderJumper_2_Open -> Jumper:SolderJumper_2_Bridged
- U2, U4: value 3V3 -> 5V
Connections:
- net GPIO23 is gone; now on net DIR_2: U1.37 (IO23)
- net +12V: now also A1.8 (VMOT), A2.8 (VMOT), C3.1, C4.1, U4.3 (IN+); no longer EMGBUT1.1 (Pin_1), U2.3 (IN+)
- net +3V3: now also J1.2 (V), J3.3 (VCC), J4.2 (V), J5.2 (V); no longer U2.1 (VO+)
- net BATTERY_INPUT: now also EMGBUT1.2 (Pin_2)
- net DIR_2: no longer U1.7 (IO32)
- net EMERGENCY_BUTTON: now also EMGBUT1.1 (Pin_1), U3.1 (VIN+); no longer A1.8 (VMOT), A2.8 (VMOT), C3.1, C4.1, EMGBUT1.2 (Pin_2), U4.3 (IN+)
- net GND: now also D1.1 (K), J1.1 (G), J3.4 (GND), J4.1 (G), J5.1 (G); no longer U1.4 (SENSOR_VN)
- net GPIO12: now also GPIO2.2 (Pin_2); no longer GPIO2.3 (Pin_3)
- net GPIO15: now also GPIO2.3 (Pin_3)
- net GPIO2: now also R4.2; no longer U5.6 (XSHUT)
- net NOT_MOT_EN: now also U1.26 (IO4); no longer U1.8 (IO33)
- net POWER_SWITCH: now also U2.3 (IN+); no longer U3.1 (VIN+)
- net SCL: now also J3.2 (SCL)
- net SDA: now also J3.1 (SDA)
- net SERVO_PWM_1: now also SRV1.6 (Pin_6); no longer SRV1.5 (Pin_5)
- net SERVO_PWM_2: now also SRV1.5 (Pin_5); no longer SRV1.6 (Pin_6)
- net at U1.19 (EXT_5V): now also D2.1 (K)
- removed net GPIO4: GPIO2.2 (Pin_2), U1.26 (IO4)
- new net: D1.2 (A), R4.1
- new net 5V_BOARD: D2.2 (A), U2.1 (VO+)
- new net TCRT0: J1.3 (S), U1.7 (IO32)
- new net TCRT1: J4.3 (S), U1.4 (SENSOR_VN)
- new net TCRT2: J5.3 (S), U1.8 (IO33)
- no-connect marks 19 -> 15
Other:
- note added: "IR"
- moved on the sheet: U5

Commit message: Fix pcb v3
Parts:
- removed GPIO2: Conn_01x07_Male, Connector_PinHeader_2.54mm:PinHeader_1x07_P2.54mm_Vertical, symbol Connector:Conn_01x07_Male
- C3, C4: footprint Capacitor_THT:CP_Radial_D4.0mm_P2.00mm -> Capacitor_THT:CP_Radial_D6.3mm_P2.50mm
Connections:
- net BATTERY_INPUT: no longer EMGBUT1.2 (Pin_2)
- net POWER_SWITCH: now also EMGBUT1.2 (Pin_2)
- net at MOT2.1 (Pin_1): now also A2.6 (2B); no longer A2.3 (1B)
- net at MOT2.2 (Pin_2): now also A2.5 (2A); no longer A2.4 (1A)
- net at MOT2.3 (Pin_3): now also A2.4 (1A); no longer A2.5 (2A)
- net at MOT2.4 (Pin_4): now also A2.3 (1B); no longer A2.6 (2B)
- net at A1.3 (1B): now also MOT1.4 (Pin_4); no longer MOT1.1 (Pin_1)
- net at A1.4 (1A): now also MOT1.3 (Pin_3); no longer MOT1.2 (Pin_2)
- net at A1.5 (2A): now also MOT1.2 (Pin_2); no longer MOT1.3 (Pin_3)
- net at A1.6 (2B): now also MOT1.1 (Pin_1); no longer MOT1.4 (Pin_4)
Other:
- moved on the sheet: MOT1, MOT2
Changed lines of the file:
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@@
     (effects (font (size 1.27 1.27)) (justify left bottom))
   )
-  (label "GPIO0" (at 233.68 39.37 0) (fields_autoplaced)
+  (label "GPIO0" (at 95.25 140.97 0) (fields_autoplaced)
     (effects (font (size 1.27 1.27)) (justify left bottom))
   )
@@
     (effects (font (size 1.27 1.27)) (justify right bottom))
   )
-  (label "GPIO35" (at 233.68 54.61 0) (fields_autoplaced)
+  (label "GPIO35" (at 20.955 116.84 0) (fields_autoplaced)
     (effects (font (size 1.27 1.27)) (justify left bottom))
   )
@@
     (effects (font (size 1.27 1.27)) (justify left bottom))
   )
-  (label "GPIO19" (at 233.68 49.53 0) (fields_autoplaced)
+  (label "GPIO19" (at 95.25 148.59 0) (fields_autoplaced)
     (effects (font (size 1.27 1.27)) (justify left bottom))
   )
@@
     (effects (font (size 1.27 1.27)) (justify right bottom))
   )
-  (label "GPIO15" (at 233.68 44.45 0) (fields_autoplaced)
+  (label "GPIO15" (at 95.25 143.51 0) (fields_autoplaced)
     (effects (font (size 1.27 1.27)) (justify left bottom))
   )
@@
     (effects (font (size 1.27 1.27)) (justify right bottom))
   )
-  (label "GPIO12" (at 233.68 41.91 0) (fields_autoplaced)
+  (label "GPIO12" (at 20.955 114.3 0) (fields_autoplaced)
     (effects (font (size 1.27 1.27)) (justify left bottom))
   )
@@
     (effects (font (size 1.27 1.27)) (justify right bottom))
   )
-  (label "BATTERY_INPUT" (at 46.99 66.04 180) (fields_autoplaced)
-    (effects (font (size 1.27 1.27)) (justify right bottom))
-  )
   (label "SERVO_PWM_2" (at 34.29 148.59 180) (fields_autoplaced)
     (effects (font (size 1.27 1.27)) (justify right bottom))
@@
     (effects (font (size 1.27 1.27)) (justify right bottom))
   )
-  (label "GPIO34" (at 233.68 52.07 0) (fields_autoplaced)
+  (label "GPIO34" (at 20.955 119.38 0) (fields_autoplaced)
     (effects (font (size 1.27 1.27)) (justify left bottom))
   )
@@
     (effects (font (size 1.27 1.27)) (justify left bottom))
   )
-  (label "GPIO18" (at 233.68 46.99 0) (fields_autoplaced)
+  (label "GPIO18" (at 95.25 146.05 0) (fields_autoplaced)
     (effects (font (size 1.27 1.27)) (justify left bottom))
   )
@@
   )
   (label "BATTERY_INPUT" (at 36.195 36.83 180) (fields_autoplaced)
+    (effects (font (size 1.27 1.27)) (justify right bottom))
+  )
+  (label "POWER_SWITCH" (at 46.99 66.04 180) (fields_autoplaced)
     (effects (font (size 1.27 1.27)) (justify right bottom))
   )
@@
       (effects (font (size 1.27 1.27)))
     )
-    (property "Footprint" "Capacitor_THT:CP_Radial_D4.0mm_P2.00mm" (at 187.96 108.2548 0)
+    (property "Footprint" "Capacitor_THT:CP_Radial_D6.3mm_P2.50mm" (at 187.96 108.2548 0)
       (effects (font (size 1.27 1.27)) hide)
     )
@@
     )
   )
-  (symbol (lib_id "Connector:Conn_01x04_Male") (at 247.65 134.62 0) (mirror y) (unit 1)
+  (symbol (lib_id "Connector:Conn_01x04_Male") (at 247.65 137.16 180) (unit 1)
     (in_bom yes) (on_board yes) (dnp no)
-    (property "Reference" "MOT2" (at 243.84 125.73 0)
+    (property "Reference" "MOT2" (at 243.84 146.05 0)
       (effects (font (size 1.27 1.27)) (justify right))
     )
-    (property "Value" "Conn_01x04_Male" (at 243.84 128.27 0)
+    (property "Value" "Conn_01x04_Male" (at 243.84 143.51 0)
       (effects (font (size 1.27 1.27)) (justify right))
     )
-    (property "Footprint" "Connector_JST:JST_SH_BM04B-SRSS-TB_1x04-1MP_P1.00mm_Vertical" (at 247.65 134.62 0)
-      (effects (font (size 1.27 1.27)) hide)
-    )
-    (property "Datasheet" "~" (at 247.65 134.62 0)
+    (property "Footprint" "Connector_JST:JST_SH_BM04B-SRSS-TB_1x04-1MP_P1.00mm_Vertical" (at 247.65 137.16 0)
+      (effects (font (size 1.27 1.27)) hide)
+    )
+    (property "Datasheet" "~" (at 247.65 137.16 0)
       (effects (font (size 1.27 1.27)) hide)
     )
@@
         (path "/25619b26-f8ce-486a-87c9-e743f43b219f"
           (reference "D2") (unit 1)
-        )
-      )
-    )
-  )
-  (symbol (lib_id "Connector:Conn_01x07_Male") (at 228.6 46.99 0) (unit 1)
-    (in_bom yes) (on_board yes) (dnp no)
-    (property "Reference" "GPIO2" (at 230.505 33.655 0)
-      (effects (font (size 1.27 1.27)))
-    )
-    (property "Value" "Conn_01x07_Male" (at 230.505 36.195 0)
-      (effects (font (size 1.27 1.27)))
-    )
-    (property "Footprint" "Connector_PinHeader_2.54mm:PinHeader_1x07_P2.54mm_Vertical" (at 228.6 46.99 0)
-      (effects (font (size 1.27 1.27)) hide)
-    )
-    (property "Datasheet" "~" (at 228.6 46.99 0)
-      (effects (font (size 1.27 1.27)) hide)
-    )
-    (pin "1")
-    (pin "2")
-    (pin "3")
-    (pin "4")
-    (pin "5")
-    (pin "6")
-    (pin "7")
-    (instances
-      (project "MiAM_PAMI_V3_Stepper"
-        (path "/25619b26-f8ce-486a-87c9-e743f43b219f"
-          (reference "GPIO2") (unit 1)
         )
       )
@@
     )
   )
-  (symbol (lib_id "Connector:Conn_01x04_Male") (at 193.04 134.62 0) (mirror y) (unit 1)
+  (symbol (lib_id "Connector:Conn_01x04_Male") (at 193.04 137.16 180) (unit 1)
     (in_bom yes) (on_board yes) (dnp no)
-    (property "Reference" "MOT1" (at 189.23 125.73 0)
+    (property "Reference" "MOT1" (at 189.23 146.05 0)
       (effects (font (size 1.27 1.27)) (justify right))
     )
-    (property "Value" "Conn_01x04_Male" (at 189.23 128.27 0)
+    (property "Value" "Conn_01x04_Male" (at 189.23 143.51 0)
       (effects (font (size 1.27 1.27)) (justify right))
     )
-    (property "Footprint" "Connector_JST:JST_SH_BM04B-SRSS-TB_1x04-1MP_P1.00mm_Vertical" (at 193.04 134.62 0)
-      (effects (font (size 1.27 1.27)) hide)
-    )
-    (property "Datasheet" "~" (at 193.04 134.62 0)
+    (property "Footprint" "Connector_JST:JST_SH_BM04B-SRSS-TB_1x04-1MP_P1.00mm_Vertical" (at 193.04 137.16 0)
+      (effects (font (size 1.27 1.27)) hide)
+    )
+    (property "Datasheet" "~" (at 193.04 137.16 0)
       (effects (font (size 1.27 1.27)) hide)
     )
@@
       (effects (font (size 1.27 1.27)))
     )
-    (property "Footprint" "Capacitor_THT:CP_Radial_D4.0mm_P2.00mm" (at 242.57 108.2548 0)
-      (effects (font (size 1.27 1.27)) hide)
-    )
+    (property "Footprint" "Capacitor_THT:CP_Radial_D6.3mm_P2.50mm" (at 242.57 108.2548 0)
+      (effects (font (size 1.27 1.27)) hide)
+    )

Commit message: PCB order 2023-11-29
Parts:
- removed R3: 10k, Resistor_SMD:R_0805_2012Metric_Pad1.20x1.40mm_HandSolder, symbol Device:R
- added J6, J7, J8: Conn_01x02_Pin, Connector_PinHeader_2.54mm:PinHeader_1x02_P2.54mm_Vertical, symbol Connector:Conn_01x02_Pin
- added J9: Conn_01x01_Pin, Connector_PinHeader_2.54mm:PinHeader_1x01_P2.54mm_Vertical, symbol Connector:Conn_01x01_Pin
- MS1, MS2, MS3: value SolderJumper_2_Bridged -> SolderJumper_2_Open; footprint Jumper:SolderJumper-2_P1.3mm_Bridged_RoundedPad1.0x1.5mm -> Jumper:SolderJumper-2_P1.3mm_Open_RoundedPad1.0x1.5mm; symbol Jumper:SolderJumper_2_Bridged -> Jumper:SolderJumper_2_Open
Connections:
- net GND: now also EMGBUT1.3 (Pin_3)
- net GPIO0: now also J8.1 (Pin_1)
- net GPIO12: now also J9.1 (Pin_1)
- net GPIO15: now also J8.2 (Pin_2)
- net GPIO18: now also J7.1 (Pin_1)
- net GPIO19: now also J7.2 (Pin_2)
- net GPIO34: now also J6.2 (Pin_2)
- net GPIO35: now also J6.1 (Pin_1)
Changed lines of the file:
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@@
     (effects (font (size 1.27 1.27)) (justify left bottom))
   )
-  (label "GPIO0" (at 95.25 140.97 0) (fields_autoplaced)
+  (label "GPIO0" (at 80.01 104.14 0) (fields_autoplaced)
     (effects (font (size 1.27 1.27)) (justify left bottom))
   )
@@
     (effects (font (size 1.27 1.27)) (justify right bottom))
   )
-  (label "GPIO35" (at 20.955 116.84 0) (fields_autoplaced)
+  (label "GPIO35" (at 26.67 115.57 0) (fields_autoplaced)
     (effects (font (size 1.27 1.27)) (justify left bottom))
   )
@@
     (effects (font (size 1.27 1.27)) (justify left bottom))
   )
-  (label "GPIO19" (at 95.25 148.59 0) (fields_autoplaced)
+  (label "GPIO19" (at 80.01 116.84 0) (fields_autoplaced)
     (effects (font (size 1.27 1.27)) (justify left bottom))
   )
@@
     (effects (font (size 1.27 1.27)) (justify right bottom))
   )
-  (label "GPIO15" (at 95.25 143.51 0) (fields_autoplaced)
+  (label "GPIO15" (at 80.01 106.68 0) (fields_autoplaced)
     (effects (font (size 1.27 1.27)) (justify left bottom))
   )
@@
     (effects (font (size 1.27 1.27)) (justify right bottom))
   )
-  (label "GPIO12" (at 20.955 114.3 0) (fields_autoplaced)
+  (label "GPIO12" (at 33.02 106.68 0) (fields_autoplaced)
     (effects (font (size 1.27 1.27)) (justify left bottom))
   )
@@
     (effects (font (size 1.27 1.27)) (justify right bottom))
   )
-  (label "GPIO34" (at 20.955 119.38 0) (fields_autoplaced)
+  (label "GPIO34" (at 26.67 118.11 0) (fields_autoplaced)
     (effects (font (size 1.27 1.27)) (justify left bottom))
   )
@@
     (effects (font (size 1.27 1.27)) (justify left bottom))
   )
-  (label "GPIO18" (at 95.25 146.05 0) (fields_autoplaced)
+  (label "GPIO18" (at 80.01 114.3 0) (fields_autoplaced)
     (effects (font (size 1.27 1.27)) (justify left bottom))
   )
@@
         (path "/25619b26-f8ce-486a-87c9-e743f43b219f"
           (reference "C3") (unit 1)
+        )
+      )
+    )
+  )
+  (symbol (lib_id "Connector:Conn_01x02_Pin") (at 74.93 104.14 0) (unit 1)
+    (in_bom yes) (on_board yes) (dnp no) (fields_autoplaced)
+    (property "Reference" "J8" (at 75.565 99.06 0)
+      (effects (font (size 1.27 1.27)))
+    )
+    (property "Value" "Conn_01x02_Pin" (at 75.565 101.6 0)
+      (effects (font (size 1.27 1.27)))
+    )
+    (property "Footprint" "Connector_PinHeader_2.54mm:PinHeader_1x02_P2.54mm_Vertical" (at 74.93 104.14 0)
+      (effects (font (size 1.27 1.27)) hide)
+    )
+    (property "Datasheet" "~" (at 74.93 104.14 0)
+      (effects (font (size 1.27 1.27)) hide)
+    )
+    (pin "2")
+    (pin "1")
+    (instances
+      (project "MiAM_PAMI_V3_Stepper"
+        (path "/25619b26-f8ce-486a-87c9-e743f43b219f"
+          (reference "J8") (unit 1)
         )
       )
@@
     )
   )
+  (symbol (lib_id "Connector:Conn_01x02_Pin") (at 74.93 114.3 0) (unit 1)
+    (in_bom yes) (on_board yes) (dnp no) (fields_autoplaced)
+    (property "Reference" "J7" (at 75.565 109.22 0)
+      (effects (font (size 1.27 1.27)))
+    )
+    (property "Value" "Conn_01x02_Pin" (at 75.565 111.76 0)
+      (effects (font (size 1.27 1.27)))
+    )
+    (property "Footprint" "Connector_PinHeader_2.54mm:PinHeader_1x02_P2.54mm_Vertical" (at 74.93 114.3 0)
+      (effects (font (size 1.27 1.27)) hide)
+    )
+    (property "Datasheet" "~" (at 74.93 114.3 0)
+      (effects (font (size 1.27 1.27)) hide)
+    )
+    (pin "2")
+    (pin "1")
+    (instances
+      (project "MiAM_PAMI_V3_Stepper"
+        (path "/25619b26-f8ce-486a-87c9-e743f43b219f"
+          (reference "J7") (unit 1)
+        )
+      )
+    )
+  )
   (symbol (lib_id "power:+12V") (at 116.84 35.56 0) (unit 1)
     (in_bom yes) (on_board yes) (dnp no)
@@
         (path "/25619b26-f8ce-486a-87c9-e743f43b219f"
           (reference "EMGBUT1") (unit 1)
+        )
+      )
+    )
+  )
+  (symbol (lib_id "Connector:Conn_01x01_Pin") (at 27.94 106.68 0) (unit 1)
+    (in_bom yes) (on_board yes) (dnp no) (fields_autoplaced)
+    (property "Reference" "J9" (at 28.575 101.6 0)
+      (effects (font (size 1.27 1.27)))
+    )
+    (property "Value" "Conn_01x01_Pin" (at 28.575 104.14 0)
+      (effects (font (size 1.27 1.27)))
+    )
+    (property "Footprint" "Connector_PinHeader_2.54mm:PinHeader_1x01_P2.54mm_Vertical" (at 27.94 106.68 0)
+      (effects (font (size 1.27 1.27)) hide)
+    )
+    (property "Datasheet" "~" (at 27.94 106.68 0)
+      (effects (font (size 1.27 1.27)) hide)
+    )
+    (pin "1")
+    (instances
+      (project "MiAM_PAMI_V3_Stepper"
+        (path "/25619b26-f8ce-486a-87c9-e743f43b219f"
+          (reference "J9") (unit 1)
         )
       )
@@
     )
   )
-  (symbol (lib_id "Jumper:SolderJumper_2_Bridged") (at 157.48 182.88 0) (unit 1)
+  (symbol (lib_id "Jumper:SolderJumper_2_Open") (at 157.48 182.88 0) (unit 1)
     (in_bom yes) (on_board yes) (dnp no) (fields_autoplaced)
     (property "Reference" "MS2" (at 157.48 176.53 0)
       (effects (font (size 1.27 1.27)))
     )
-    (property "Value" "SolderJumper_2_Bridged" (at 157.48 179.07 0)
-      (effects (font (size 1.27 1.27)))
-    )
-    (property "Footprint" "Jumper:SolderJumper-2_P1.3mm_Bridged_RoundedPad1.0x1.5mm" (at 157.48 182.88 0)
+    (property "Value" "SolderJumper_2_Open" (at 157.48 179.07 0)
+      (effects (font (size 1.27 1.27)))
+    )
+    (property "Footprint" "Jumper:SolderJumper-2_P1.3mm_Open_RoundedPad1.0x1.5mm" (at 157.48 182.88 0)
       (effects (font (size 1.27 1.27)) hide)
     )
@@
     )
   )
-  (symbol (lib_id "Device:R") (at 43.18 68.58 90) (unit 1)
-    (in_bom yes) (on_board yes) (dnp no)
-    (property "Reference" "R3" (at 43.815 71.755 90)
-      (effects (font (size 1.27 1.27)))
-    )
-    (property "Value" "10k" (at 43.815 74.295 90)
-      (effects (font (size 1.27 1.27)))
-    )
-    (property "Footprint" "Resistor_SMD:R_0805_2012Metric_Pad1.20x1.40mm_HandSolder" (at 43.18 70.358 90)
-      (effects (font (size 1.27 1.27)) hide)
-    )
-    (property "Datasheet" "~" (at 43.18 68.58 0)
-      (effects (font (size 1.27 1.27)) hide)
-    )
-    (pin "1")
-    (pin "2")
-    (instances
-      (project "MiAM_PAMI_V3_Stepper"
-        (path "/25619b26-f8ce-486a-87c9-e743f43b219f"
-          (reference "R3") (unit 1)
-        )
-      )
-    )
-  )
   (symbol (lib_id "power:+12V") (at 234.95 105.41 0) (unit 1)
     (in_bom yes) (on_board yes) (dnp no)
@@
     )
   )
-  (symbol (lib_id "Jumper:SolderJumper_2_Bridged") (at 157.48 173.99 0) (unit 1)
+  (symbol (lib_id "Jumper:SolderJumper_2_Open") (at 157.48 173.99 0) (unit 1)
     (in_bom yes) (on_board yes) (dnp no) (fields_autoplaced)
     (property "Reference" "MS1" (at 157.48 167.64 0)
       (effects (font (size 1.27 1.27)))
     )
-    (property "Value" "SolderJumper_2_Bridged" (at 157.48 170.18 0)
-      (effects (font (size 1.27 1.27)))
-    )
-    (property "Footprint" "Jumper:SolderJumper-2_P1.3mm_Bridged_RoundedPad1.0x1.5mm" (at 157.48 173.99 0)
+    (property "Value" "SolderJumper_2_Open" (at 157.48 170.18 0)
+      (effects (font (size 1.27 1.27)))
+    )
+    (property "Footprint" "Jumper:SolderJumper-2_P1.3mm_Open_RoundedPad1.0x1.5mm" (at 157.48 173.99 0)
       (effects (font (size 1.27 1.27)) hide)
     )
@@
         (path "/25619b26-f8ce-486a-87c9-e743f43b219f"
           (reference "#PWR0120") (unit 1)
+        )
+      )
+    )
+  )
+  (symbol (lib_id "Connector:Conn_01x02_Pin") (at 21.59 115.57 0) (unit 1)
+    (in_bom yes) (on_board yes) (dnp no) (fields_autoplaced)
+    (property "Reference" "J6" (at 22.225 110.49 0)
+      (effects (font (size 1.27 1.27)))
+    )
+    (property "Value" "Conn_01x02_Pin" (at 22.225 113.03 0)
+      (effects (font (size 1.27 1.27)))
+    )
+    (property "Footprint" "Connector_PinHeader_2.54mm:PinHeader_1x02_P2.54mm_Vertical" (at 21.59 115.57 0)
+      (effects (font (size 1.27 1.27)) hide)
+    )
+    (property "Datasheet" "~" (at 21.59 115.57 0)
+      (effects (font (size 1.27 1.27)) hide)
+    )
+    (pin "2")
+    (pin "1")
+    (instances
+      (project "MiAM_PAMI_V3_Stepper"
+        (path "/25619b26-f8ce-486a-87c9-e743f43b219f"
+          (reference "J6") (unit 1)
         )
       )
@@
     )
   )
-  (symbol (lib_id "Jumper:SolderJumper_2_Bridged") (at 157.48 191.77 0) (unit 1)
+  (symbol (lib_id "Jumper:SolderJumper_2_Open") (at 157.48 191.77 0) (unit 1)
     (in_bom yes) (on_board yes) (dnp no) (fields_autoplaced)
     (property "Reference" "MS3" (at 157.48 185.42 0)
       (effects (font (size 1.27 1.27)))
     )
-    (property "Value" "SolderJumper_2_Bridged" (at 157.48 187.96 0)
-      (effects (font (size 1.27 1.27)))
-    )
-    (property "Footprint" "Jumper:SolderJumper-2_P1.3mm_Bridged_RoundedPad1.0x1.5mm" (at 157.48 191.77 0)
+    (property "Value" "SolderJumper_2_Open" (at 157.48 187.96 0)
+      (effects (font (size 1.27 1.27)))
+    )
+    (property "Footprint" "Jumper:SolderJumper-2_P1.3mm_Open_RoundedPad1.0x1.5mm" (at 157.48 191.77 0)
       (effects (font (size 1.27 1.27)) hide)
     )
@@
     )
   )
-  (symbol (lib_id "power:GND") (at 39.37 68.58 0) (unit 1)
-    (in_bom yes) (on_board yes) (dnp no) (fields_autoplaced)
-    (property "Reference" "#PWR023" (at 39.37 74.93 0)
-      (effects (font (size 1.27 1.27)) hide)
-    )
-    (property "Value" "GND" (at 39.37 73.66 0)
-      (effects (font (size 1.27 1.27)))
-    )
-    (property "Footprint" "" (at 39.37 68.58 0)
-      (effects (font (size 1.27 1.27)) hide)
-    )
-    (property "Datasheet" "" (at 39.37 68.58 0)
-      (effects (font (size 1.27 1.27)) hide)
-    )
+  (symbol (lib_id "power:GND") (at 46.99 68.58 0) (unit 1)
+    (in_bom yes) (on_board yes) (dnp no) (fields_autoplaced)
+    (property "Reference" "#PWR023" (at 46.99 74.93 0)
+      (effects (font (size 1.27 1.27)) hide)
+    )
+    (property "Value" "GND" (at 46.99 73.66 0)
+      (effects (font (size 1.27 1.27)))
+    )
+    (property "Footprint" "" (at 46.99 68.58 0)
+      (effects (font (size 1.27 1.27)) hide)
+    )
+    (property "Datasheet" "" (at 46.99 68.58 0)
+      (effects (font (size 1.27 1.27)) hide)
+    )
